File: rfidLock3/rfidLock3.brd (EAGLE design)
At the start: 99.7 x 83.2 mm, 53 parts, among them IC1 ATMEGA328, SW1 TPK, SW10 TPK, SW11 TPK, SW12 TPK, SW13 TPK, SW14 TPK, SW15 TPK, SW16 TPK, SW2 TPK, SW3 TPK, SW4 TPK, SW5 TPK, SW6 TPK, SW7 TPK, SW8 TPK, SW9 TPK, Y1 16MHz

Commit message: pcb update
Parts:
- added U$1: ESP8266-07, lio:ESP-07
- JP1: device pinhead:1X08 -> pinhead:1X04
- moved R9 120.6 mm to (64.8, 73.0), turned to 180 degrees
- moved R8 120.6 mm to (64.8, 71.1), turned to 180 degrees
- moved R5 111.5 mm to (47.0, 77.2)
- moved R7 107.8 mm to (7.62, 78.7)
- moved R6 105.3 mm to (7.62, 76.5)
- moved C5 101.9 mm to (13.3, 73.0), turned to 90 degrees
- moved C3 101.3 mm to (18.7, 78.4), turned to 45 degrees
- moved C4 98.6 mm to (31.8, 65.4), turned to 180 degrees
- moved Y1 97.4 mm to (16.5, 72.4), turned to 90 degrees
- moved C6 97.2 mm to (16.5, 68.3)
- moved LED18 97.2 mm to (3.81, 78.7), turned to 90 degrees
- moved C7 94.4 mm to (20.6, 77.2), turned to 45 degrees
- moved LED13 92.9 mm to (95.2, 55.2), turned to 0 degrees
- moved LED17 82.2 mm to (3.81, 76.5), turned to 90 degrees
- moved LED9 72.9 mm to (80.0, 55.2), turned to 0 degrees
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Connections:
- net N$24 renamed CRYSTAL1
- net N$25 renamed CRYSTAL2
- removed net N$11: JP1.2
- removed net N$5 (its old number): JP1.8
- net +3V3: now also JP1.4, U$1.VCC; no longer JP1.1
- net +5V: now also C3.1, JP1.1; no longer C3.2
- net A0: now also SW13.2, SW14.2, SW15.2, SW16.2; no longer SW1.1, SW13.1, SW5.1, SW9.1
- net A2: now also SW5.2, SW6.2, SW7.2, SW8.2; no longer SW11.1, SW15.1, SW3.1, SW7.1
- net A3: now also SW11.1, SW15.1, SW3.1, SW7.1; no longer SW12.1, SW16.1, SW4.1, SW8.1
- net A5: now also SW12.1, SW16.1, SW4.1, SW8.1; no longer SW5.2, SW6.2, SW7.2, SW8.2
- net A6: now also SW1.1, SW13.1, SW5.1, SW9.1; no longer SW10.2, SW11.2, SW12.2, SW9.2
- net A7: now also SW10.2, SW11.2, SW12.2, SW9.2; no longer SW13.2, SW14.2, SW15.2, SW16.2
- net D11: no longer JP1.6
- net D12: no longer JP1.5
- net D13: no longer JP1.7
- net GND: now also C3.2, JP1.2, U$1.GND; no longer C3.1
Routing:
- net A0: track 45.8 -> 141.3 mm
- net A7: track 35.6 -> 128.3 mm, vias 7 -> 6
- net A5: track 34.9 -> 121.6 mm, vias 7 -> 0
- net A4: track 43.8 -> 125.4 mm, vias 9 -> 6
- net +5V: track 0.00 -> 65.8 mm, vias 0 -> 1
- net A2: track 65.5 -> 130.1 mm, vias 3 -> 6
- net N$2: track 0.00 -> 63.9 mm
- net N$3: track 0.00 -> 56.1 mm
- net N$1: track 0.00 -> 53.6 mm
- net N$4: track 0.00 -> 45.8 mm
- net A3: track 64.8 -> 103.9 mm, vias 7 -> 0
- net D1/TX: track 0.00 -> 38.7 mm
- net D0/RX: track 0.00 -> 38.7 mm
- net A6: track 38.8 -> 74.0 mm, vias 7 -> 0
- net A1: track 57.2 -> 83.6 mm, vias 1 -> 0
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Other:
- board size 99.7 x 83.2 mm -> 101.6 x 81.3 mm

Commit message: update
Parts:
- added Q1: BSS123, transistor-small-signal:SOT23
- added R10: 1k, SparkFun:0603-RES
- moved LED17 40.5 mm to (40.6, 59.7), turned to 270 degrees
- moved R1 34.2 mm to (55.9, 14.0), turned to 90 degrees
- moved R6 33.7 mm to (36.8, 59.7), turned to 180 degrees
- moved C2 15.4 mm to (65.4, 72.4)
- moved R5 12.1 mm to (59.1, 77.2)
- moved LED18 5.08 mm to (8.89, 78.7)
- moved R7 5.08 mm to (12.7, 78.7)
- moved C3 3.55 mm to (15.6, 76.8), turned to 180 degrees
- moved U$1 3.00 mm to (86.4, 76.5)
- moved JP1 2.71 mm to (66.0, 77.8)
- moved R8 2.62 mm to (65.4, 68.6)
- moved R9 2.62 mm to (65.4, 70.5)
- moved C4 1.31 mm to (33.0, 65.1)
- moved R2 0.63 mm to (73.0, 14.0)
Connections:
- new net LGND: LED1.C, LED10.C, LED11.C, LED12.C, LED13.C, LED14.C, LED15.C, LED16.C, LED2.C, LED3.C, LED4.C, LED5.C, LED6.C, LED7.C, LED8.C, LED9.C, Q1.3
- new net LPWM: Q1.1, R10.1
- net A2: no longer SW5.2, SW6.2, SW7.2, SW8.2
- net D3: now also R10.2
- net D4: now also SW5.2, SW6.2, SW7.2, SW8.2
- net GND: now also Q1.2; no longer LED1.C, LED10.C, LED11.C, LED12.C, LED13.C, LED14.C, LED15.C, LED16.C, LED2.C, LED3.C, LED4.C, LED5.C, LED6.C, LED7.C, LED8.C, LED9.C
Routing:
- net D4: track 0.00 -> 140.6 mm, vias 0 -> 8
- net A2: track 130.1 -> 0.00 mm, vias 6 -> 0
- net +3V3: track 0.97 -> 115.7 mm, vias 0 -> 8
- net D3: track 0.00 -> 72.9 mm, vias 0 -> 4
- net RESET: track 22.2 -> 41.0 mm
- net D13: track 0.00 -> 11.7 mm
- net +5V: track 65.8 -> 76.1 mm, vias 1 -> 2
- net N$4: track 45.8 -> 53.6 mm
- net A0: track 141.3 -> 148.4 mm
- net A7: track 128.3 -> 132.4 mm
- net A1: track 83.6 -> 87.6 mm
- net LPWM: track 0.00 -> 2.81 mm
- net A5: track 121.6 -> 119.7 mm
- net D1/TX: track 38.7 -> 40.4 mm
- net D0/RX: track 38.7 -> 40.4 mm
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- added copper zone on layer 1, net LGND

Commit message: another update
Parts:
- added JP2: (no value), pinhead:1X08
- added R11: 1k, SparkFun:0805
- C2, C3, C4, C5, C6: device SparkFun:0603-CAP -> SparkFun:0805
- R1, R2, R3, R4: value (none) -> 1k; device resistor:M1206 -> SparkFun:0805
- R10, R5, R6, R7, R8, R9: device SparkFun:0603-RES -> SparkFun:0805
- moved R10 28.9 mm to (61.3, 61.0)
- moved Q1 22.0 mm to (68.6, 60.0), turned to 270 degrees
- moved R5 14.9 mm to (44.1, 77.2), turned to 180 degrees
- moved R6 5.62 mm to (40.6, 63.8), turned to 0 degrees
- moved LED17 5.41 mm to (37.1, 63.8), turned to 90 degrees
- moved LED18 4.55 mm to (13.3, 77.8), turned to 180 degrees
- moved R7 3.81 mm to (16.5, 78.7)
- moved C2 2.03 mm to (67.0, 73.7)
- moved R8 2.03 mm to (67.0, 69.8)
- moved R9 2.03 mm to (67.0, 71.8)
- moved C4 1.27 mm to (33.0, 63.8)
- moved C3 1.00 mm to (16.5, 76.5)
- moved C5 0.95 mm to (13.3, 74.0), turned to 270 degrees
- moved JP1 0.63 mm to (66.7, 77.8)
- moved R2 0.63 mm to (73.7, 14.0), turned to 270 degrees
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Connections:
- removed net A6: IC1.19, SW1.1, SW13.1, SW5.1, SW9.1
- removed net D10: IC1.14
- removed net D11: IC1.15
- removed net D12: IC1.16
- removed net D13: IC1.17, R6.2
- new net IRQ: JP2.5
- new net MISO: IC1.16, JP2.4
- new net MOSI: IC1.15, JP2.3
- new net RST: IC1.14, JP2.7
- new net SCK: IC1.17, JP2.2, R6.2
- new net SDA: IC1.19, JP2.1
- net +3V3: now also JP2.8, R1.1, R2.1, R3.1, R4.1; no longer R1.2, R2.2, R3.2, R4.2
- net A0: now also SW10.2, SW11.2, SW12.2, SW9.2; no longer SW13.2, SW14.2, SW15.2, SW16.2
- net A1: now also SW13.2, SW14.2, SW15.2, SW16.2; no longer SW10.1, SW14.1, SW2.1, SW6.1
- net A7: now also SW1.1, SW13.1, SW5.1, SW9.1; no longer SW10.2, SW11.2, SW12.2, SW9.2
- net D5: now also SW10.1, SW14.1, SW2.1, SW6.1
- net GND: now also JP2.6, R11.2
- net LPWM: now also R11.1
- net N$1: now also R3.2; no longer R3.1
- net N$2: now also R4.2; no longer R4.1
- net N$3: now also R2.2; no longer R2.1
- net N$4: now also R1.2; no longer R1.1
Routing:
- net D5: track 0.00 -> 99.2 mm, vias 0 -> 2
- net A6: track 75.5 -> 0.00 mm
- net A1: track 87.6 -> 146.8 mm
- net A7: track 132.4 -> 76.0 mm, vias 6 -> 0
- net +3V3: track 115.7 -> 169.5 mm, vias 8 -> 10
- net D3: track 72.9 -> 43.2 mm, vias 4 -> 2
- net SCK: track 0.00 -> 21.9 mm, vias 0 -> 2
- net A0: track 148.4 -> 131.3 mm, vias 0 -> 6
- net D13: track 11.7 -> 0.00 mm
- net RST: track 0.00 -> 11.1 mm
- net LPWM: track 2.81 -> 9.75 mm
- net MOSI: track 0.00 -> 6.91 mm
- net SDA: track 0.00 -> 6.52 mm
- net +5V: track 76.1 -> 70.9 mm
- net MISO: track 0.00 -> 4.81 mm
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
Commit message: update again
Parts:
- moved C6 4.07 mm to (13.3, 70.8), turned to 90 degrees
- moved R5 1.27 mm to (42.9, 77.2)
- moved C7 0.45 mm to (21.0, 76.8)
- moved R11 0.32 mm to (61.3, 63.2)
Connections:
- net D5: no longer SW10.1, SW14.1, SW2.1, SW6.1
- net D7: now also SW10.1, SW14.1, SW2.1, SW6.1
Routing:
- net D5: track 99.2 -> 0.04 mm, vias 2 -> 0
- net D7: track 0.00 -> 96.0 mm, vias 0 -> 2
- net CRYSTAL2: track 5.24 -> 9.25 mm
- net D4: track 140.6 -> 139.7 mm
- net +5V: track 70.9 -> 70.3 mm
- net +3V3: track 169.5 -> 170.1 mm, vias 10 -> 8
- net A5: track 119.2 -> 119.7 mm

Commit message: +led, +conectors...
Parts:
- added FOTO, FOTO1, GND, SPKR: (no value), pinhead:1X01
- added LED19: LED-TRICOLOR-5050NO_IC, SparkFun-LED:LED-TRICOLOR-5050
- added R12, R13, R14, R15, R16: 1k, SparkFun:0805
- moved R5 14.3 mm to (28.6, 77.5)
- moved R2 4.44 mm to (69.2, 14.0)
- moved R4 3.49 mm to (85.4, 14.0)
- moved R3 2.86 mm to (83.5, 14.0)
- moved R1 1.59 mm to (54.3, 14.0)
- moved U$1 1.27 mm to (85.1, 76.5)
Connections:
- new net N$10: R15.1, SPKR.1
- new net N$6: LED19.1, R13.1
- new net N$8: LED19.2, R14.1
- new net N$9: LED19.3, R12.1
- net +5V: now also FOTO.1
- net A2: now also FOTO1.1, R16.1
- net D5: now also R14.2
- net D6: now also R13.2
- net D8: now also R15.2
- net D9: now also R12.2
- net GND: now also GND.1, LED19.4, LED19.5, LED19.6, R16.2
Routing:
- net A2: track 0.00 -> 46.2 mm, vias 0 -> 1
- net D9: track 0.00 -> 18.4 mm
- net N$10: track 0.00 -> 15.6 mm
- net D8: track 0.00 -> 14.8 mm
- net D6: track 0.00 -> 14.2 mm
- net D5: track 0.04 -> 11.8 mm
- net N$9: track 0.00 -> 7.02 mm
- net N$8: track 0.00 -> 5.03 mm
- net N$3: track 56.1 -> 51.6 mm
- net +3V3: track 170.1 -> 166.5 mm
- net N$2: track 64.4 -> 67.3 mm
- net N$1: track 53.5 -> 50.6 mm
- net N$6: track 0.00 -> 2.55 mm
- net N$4: track 53.5 -> 51.9 mm
- net RESET: track 42.0 -> 43.4 mm
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
Commit message: almost final version
Parts:
- removed Q1: BSS123, transistor-small-signal:SOT23
- added JP10, JP11, JP12, JP13, JP14, JP15, JP3, JP4, JP5, JP6, JP7, JP8, JP9: (no value), pinhead:1X01
- added Q2, Q3, Q4, Q5: BSS138, SparkFun:SOT23-3
- added R17, R18, R19, R20, R21, R22, R23, R24, R25, R26, R27, R28: 1k, SparkFun:0805
- added S2: TEMPER, SparkFun:TACTILE_SWITCH_SMD
- moved R16 18.2 mm to (48.9, 78.7), turned to 0 degrees
- moved R8 14.8 mm to (52.4, 67.3)
- moved R9 14.7 mm to (52.4, 69.8)
- moved C2 14.7 mm to (52.4, 72.4)
- moved R11 7.75 mm to (54.9, 58.7)
- moved FOTO1 7.30 mm to (46.0, 78.7)
- moved FOTO 7.30 mm to (43.5, 78.7)
- moved R10 6.35 mm to (54.9, 61.0)
- moved LED10 2.54 mm to (77.5, 40.0)
- moved LED11 2.54 mm to (77.5, 24.8)
- moved LED12 2.54 mm to (77.5, 9.53)
- moved LED13 2.54 mm to (92.7, 55.2)
- moved LED14 2.54 mm to (92.7, 40.0)
- moved LED15 2.54 mm to (92.7, 24.8)
- moved LED16 2.54 mm to (92.7, 9.53)
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Connections:
- new net DTR_OUT: JP13.1, Q4.2, R26.1, U$1.GPIO16
- new net HV1: JP7.1, Q2.3, R23.1
- new net HV2: JP8.1, Q3.3, R25.1
- new net HV3: JP11.1, Q4.3, R27.1
- new net LV1: JP12.1, Q2.2, R22.1, U$1.TXD
- new net LV2: JP6.1, Q3.2, R24.1, U$1.RXD
- new net N$11: R17.2, U$1.GPIO0
- new net N$12: JP14.1, R18.2, U$1.GPIO2
- new net N$13: R19.2, U$1.GPIO15
- new net N$14: R20.2, U$1.CH_PD
- new net N$15: JP10.1, R21.2, U$1.REST
- new net N$20: R28.2, S2.3
- new net N$21: S2.4, U$1.GPIO13
- net +3V3: now also Q2.1, Q3.1, Q4.1, R17.1, R18.1, R21.1, R22.2, R24.2, R26.2, R28.1
- net +5V: now also R23.2, R25.2, R27.2
- net D0: now also JP4.1
- net D1: now also JP5.1
- net DTR: now also JP3.1
- net GND: now also JP15.1, Q5.2, R19.1, R20.1, S2.1, S2.2; no longer Q1.2
- net LGND: now also Q5.3; no longer Q1.3
- net LPWM: now also Q5.1; no longer Q1.1
- net RESET: now also JP9.1
Routing:
- net +3V3: track 166.5 -> 202.3 mm, vias 8 -> 9
- net LV1: track 0.00 -> 35.5 mm, vias 0 -> 1
- net LV2: track 0.00 -> 35.5 mm, vias 0 -> 1
- net N$15: track 0.00 -> 30.8 mm
- net N$12: track 0.00 -> 24.6 mm
- net A2: track 46.2 -> 23.3 mm
- net N$11: track 0.00 -> 15.7 mm
- net N$14: track 0.00 -> 15.2 mm
- net +5V: track 70.8 -> 85.2 mm, vias 2 -> 4
- net D1/TX: track 41.4 -> 27.6 mm
- net D0/RX: track 41.4 -> 27.8 mm
- net DTR_OUT: track 0.00 -> 12.5 mm
- net N$21: track 0.00 -> 11.1 mm, vias 0 -> 2
- net N$13: track 0.00 -> 7.43 mm
- net D3: track 43.2 -> 36.9 mm
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- added copper zone on layer 16, net GND
- added copper zone on layer 16, net LGND
Other:
- board size 101.6 x 81.3 mm -> 99.1 x 81.3 mm
