File: rfidLock3/rfidLock3.sch (EAGLE design)
At the start: 53 parts, among them IC1 ATMEGA328, SW1 TPK, SW10 TPK, SW11 TPK, SW12 TPK, SW13 TPK, SW14 TPK, SW15 TPK, SW16 TPK, SW2 TPK, SW3 TPK, SW4 TPK, SW5 TPK, SW6 TPK, SW7 TPK, SW8 TPK, SW9 TPK, Y1 16MHz

Commit message: pcb update
Parts:
- added U$1: ESP8266-07, lio:ESP8266-07
- JP1: device pinhead:PINHD-1X8 -> pinhead:PINHD-1X4
Connections:
- net N$24 renamed CRYSTAL1
- net N$25 renamed CRYSTAL2
- removed net N$11: JP1.2
- removed net N$5 (its old number): JP1.8
- net +3V3: now also JP1.4, U$1.VCC; no longer JP1.1
- net +5V: now also C3.1, JP1.1; no longer C3.2
- net A0: now also SW13.S, SW14.S, SW15.S, SW16.S; no longer SW1.P, SW13.P, SW5.P, SW9.P
- net A2: now also SW5.S, SW6.S, SW7.S, SW8.S; no longer SW11.P, SW15.P, SW3.P, SW7.P
- net A3: now also SW11.P, SW15.P, SW3.P, SW7.P; no longer SW12.P, SW16.P, SW4.P, SW8.P
- net A5: now also SW12.P, SW16.P, SW4.P, SW8.P; no longer SW5.S, SW6.S, SW7.S, SW8.S
- net A6: now also SW1.P, SW13.P, SW5.P, SW9.P; no longer SW10.S, SW11.S, SW12.S, SW9.S
- net A7: now also SW10.S, SW11.S, SW12.S, SW9.S; no longer SW13.S, SW14.S, SW15.S, SW16.S
- net D11: no longer JP1.6
- net D12: no longer JP1.5
- net D13: no longer JP1.7
- net GND: now also C3.2, JP1.2, U$1.GND; no longer C3.1
Other:
- moved on the sheet: C2, C3, C4, C5, C6, C7, IC1, LED17, LED18, R5, R6, R7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

Commit message: update
Parts:
- added Q1: BSS123, transistor-small-signal:BSS123
- added R10: 1k, SparkFun:RESISTOR0603-RES
Connections:
- new net LGND: LED1.C, LED10.C, LED11.C, LED12.C, LED13.C, LED14.C, LED15.C, LED16.C, LED2.C, LED3.C, LED4.C, LED5.C, LED6.C, LED7.C, LED8.C, LED9.C, Q1.D
- new net LPWM: Q1.G, R10.1
- net A2: no longer SW5.S, SW6.S, SW7.S, SW8.S
- net D3: now also R10.2
- net D4: now also SW5.S, SW6.S, SW7.S, SW8.S
- net GND: now also Q1.S; no longer LED1.C, LED10.C, LED11.C, LED12.C, LED13.C, LED14.C, LED15.C, LED16.C, LED2.C, LED3.C, LED4.C, LED5.C, LED6.C, LED7.C, LED8.C, LED9.C

Commit message: another update
Parts:
- added JP2: (no value), pinhead:PINHD-1X8
- added R11: 1k, SparkFun:RESISTOR0805-RES
- C2, C3, C4, C5, C6: device SparkFun:CAP0603-CAP -> SparkFun:CAP0805
- R1, R2, R3, R4: value (none) -> 1k; device resistor:R-EU_M1206 -> SparkFun:RESISTOR0805-RES
- R10, R5, R6, R7, R8, R9: device SparkFun:RESISTOR0603-RES -> SparkFun:RESISTOR0805-RES
Connections:
- removed net A6: IC1.ADC6, SW1.P, SW13.P, SW5.P, SW9.P
- removed net D10: IC1.PB2(SS/OC1B)
- removed net D11: IC1.PB3(MOSI/OC2)
- removed net D12: IC1.PB4(MISO)
- removed net D13: IC1.PB5(SCK), R6.2
- new net IRQ: JP2.5
- new net MISO: IC1.PB4(MISO), JP2.4
- new net MOSI: IC1.PB3(MOSI/OC2), JP2.3
- new net RST: IC1.PB2(SS/OC1B), JP2.7
- new net SCK: IC1.PB5(SCK), JP2.2, R6.2
- new net SDA: IC1.ADC6, JP2.1
- net +3V3: now also JP2.8, R1.1, R2.1, R3.1, R4.1; no longer R1.2, R2.2, R3.2, R4.2
- net A0: now also SW10.S, SW11.S, SW12.S, SW9.S; no longer SW13.S, SW14.S, SW15.S, SW16.S
- net A1: now also SW13.S, SW14.S, SW15.S, SW16.S; no longer SW10.P, SW14.P, SW2.P, SW6.P
- net A7: now also SW1.P, SW13.P, SW5.P, SW9.P; no longer SW10.S, SW11.S, SW12.S, SW9.S
- net D5: now also SW10.P, SW14.P, SW2.P, SW6.P
- net GND: now also JP2.6, R11.2
- net LPWM: now also R11.1
- net N$1: now also R3.2; no longer R3.1
- net N$2: now also R4.2; no longer R4.1
- net N$3: now also R2.2; no longer R2.1
- net N$4: now also R1.2; no longer R1.1
Other:
- moved on the sheet: LED18, R7

Commit message: update again
Connections:
- net D5: no longer SW10.P, SW14.P, SW2.P, SW6.P
- net D7: now also SW10.P, SW14.P, SW2.P, SW6.P
Other:
- moved on the sheet: C4, C5, C6, LED1, LED10, LED11, LED12, LED13, LED14, LED15, LED16, LED2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

Commit message: +led, +conectors...
Parts:
- added FOTO, FOTO1, GND, SPKR: (no value), pinhead:PINHD-1X1
- added LED19: LED-TRICOLOR-5050NO_IC, SparkFun-LED:LED-TRICOLOR-5050NO_IC
- added R12, R13, R14, R15, R16: 1k, SparkFun:RESISTOR0805-RES
Connections:
- new net N$10: R15.1, SPKR.1
- new net N$6: LED19.GRN-A, R13.1
- new net N$8: LED19.RED-A, R14.1
- new net N$9: LED19.BLU-A, R12.1
- net +5V: now also FOTO.1
- net A2: now also FOTO1.1, R16.1
- net D5: now also R14.2
- net D6: now also R13.2
- net D8: now also R15.2
- net D9: now also R12.2
- net GND: now also GND.1, LED19.BLU-C, LED19.GRN-C, LED19.RED-C, R16.2
Other:
- moved on the sheet: C2, C3, C4, C5, C6, C7, IC1, JP1, JP2, LED1, LED10, LED11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

Commit message: almost final version
Parts:
- removed Q1: BSS123, transistor-small-signal:BSS123
- added JP10, JP11, JP12, JP13, JP14, JP15, JP3, JP4, JP5, JP6, JP7, JP8, JP9: (no value), pinhead:PINHD-1X1
- added Q2, Q3, Q4, Q5: BSS138, SparkFun:MOSFET-NCHANNELSMD
- added R17, R18, R19, R20, R21, R22, R23, R24, R25, R26, R27, R28: 1k, SparkFun:RESISTOR0805-RES
- added S2: TEMPER, SparkFun:TAC_SWITCHSMD
Connections:
- new net DTR_OUT: JP13.1, Q4.S, R26.1, U$1.GPIO16
- new net HV1: JP7.1, Q2.D, R23.1
- new net HV2: JP8.1, Q3.D, R25.1
- new net HV3: JP11.1, Q4.D, R27.1
- new net LV1: JP12.1, Q2.S, R22.1, U$1.TXD
- new net LV2: JP6.1, Q3.S, R24.1, U$1.RXD
- new net N$11: R17.2, U$1.GPIO0
- new net N$12: JP14.1, R18.2, U$1.GPIO2
- new net N$13: R19.2, U$1.GPIO15
- new net N$14: R20.2, U$1.CH_PD
- new net N$15: JP10.1, R21.2, U$1.REST
- new net N$20: R28.2, S2.3
- new net N$21: S2.4, U$1.GPIO13
- net +3V3: now also Q2.G, Q3.G, Q4.G, R17.1, R18.1, R21.1, R22.2, R24.2, R26.2, R28.1
- net +5V: now also R23.2, R25.2, R27.2
- net D0: now also JP4.1
- net D1: now also JP5.1
- net DTR: now also JP3.1
- net GND: now also JP15.1, Q5.S, R19.1, R20.1, S2.1, S2.2; no longer Q1.S
- net LGND: now also Q5.D; no longer Q1.D
- net LPWM: now also Q5.G; no longer Q1.G
- net RESET: now also JP9.1
Other:
- moved on the sheet: C2, R16, R8, R9, U$1
